Commit message: Se corrige error de espacons en el .xacro y en el twiststam en .yaml

File: my_robot_description/urdf/mobile_base.ros2_control.xacro (robot description, xacro)
@@ -3,17 +3,13 @@
     <ros2_control name="MobileBaseHardwareInterface" type="system">
         <hardware>
-            <plugin>
-                mock_components/GenericSystem
-            </plugin>
-            <param name="calculate_dynamics">
-                true
-            </param>
+            <plugin>mock_components/GenericSystem</plugin>
+            <param name="calculate_dynamics">true</param>
         </hardware>
-        <joint name="base_right_wheel_joint" type="continuous">
+        <joint name="base_right_wheel_joint">
             <command_interface name="velocity" />
             <state_interface name="position"/>
             <state_interface name="velocity"/>
         </joint>
-        <joint name="base_left_wheel_joint" type="continuous">
+        <joint name="base_left_wheel_joint">
             <command_interface name="velocity" />
             <state_interface name="position"/>
